File: PCB/level_shifter_sch.kicad_sch (KiCad schematic)
At the start: 15 parts, among them U101 TLV9151, U102 TLV9151, U103 TLV9151, U104 TLV9151

Commit message: Intial commit
Connections:
- net +5V: now also U101.6 (V+), U102.6 (V+), U103.6 (V+), U104.6 (V+); no longer U101.4 (V+), U102.4 (V+), U103.4 (V+), U104.4 (V+)
- net GND: now also U101.3 (+), U102.3 (+), U103.3 (+), U104.3 (+); no longer U101.5 (-), U102.5 (-), U103.5 (-), U104.5 (-)
- net at R119.2, R120.2, R121.1: now also U104.4 (-); no longer U104.3 (+)
- net at R116.2, R117.2, R118.1: now also U103.4 (-); no longer U103.3 (+)
- net at R111.2, R112.2, R114.1: now also U101.4 (-); no longer U101.3 (+)
- net at R113.2, R115.1: now also U102.4 (-); no longer U102.3 (+)
Other:
- moved on the sheet: R116, R117, R118, U103
