File: PCB/rlc_meter.kicad_pcb (KiCad board)
At the start: 2 copper layers, 78.5 x 74.9 mm, 72 parts, among them IC101 STM32G431K6T6, IC102 LDL1117S33R, IC103 TPS65133DPDR, J101 571-0100, J102 Conn_01x04_Female, J103 PJ-036BH-SMT-TR, J104 Conn_01x04_Female, J105 571-0100, K101 UB2-3NU, K102 UB2-3NU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

Commit message: Intial commit
Connections:
- U101 pad 3: Net-(R111-Pad2) -> GND
- U101 pad 4: +5V -> Net-(R111-Pad2)
- U101 pad 5: GND -> (no net)
- U101 pad 6: (no net) -> +5V
- U102 pad 3: Net-(R113-Pad2) -> GND
- U102 pad 4: +5V -> Net-(R113-Pad2)
- U102 pad 5: GND -> (no net)
- U102 pad 6: (no net) -> +5V
- U103 pad 3: Net-(R116-Pad2) -> GND
- U103 pad 4: +5V -> Net-(R116-Pad2)
- U103 pad 5: GND -> (no net)
- U103 pad 6: (no net) -> +5V
- U104 pad 3: Net-(R119-Pad2) -> GND
- U104 pad 4: +5V -> Net-(R119-Pad2)
- U104 pad 5: GND -> (no net)
- U104 pad 6: (no net) -> +5V
Routing:
- net GND: track 128.6 -> 158.7 mm, vias 12 -> 14
- net Net-(R113-Pad2): track 10.4 -> 16.4 mm
- net Net-(R119-Pad2): track 22.5 -> 27.0 mm
- net Net-(R111-Pad2): track 22.0 -> 25.7 mm
- net Net-(R116-Pad2): track 22.1 -> 25.2 mm
- net +5V: track 61.7 -> 59.5 mm
Other:
- board text added: "RLC Meter v1.1 Author: Mikolaj Harazin"
- board text removed: "RLC Meter v1.0 Author: Mikolaj Harazin"
